File: gant.kicad_pcb (KiCad board)
At the start: 2 copper layers, 2 x 5.6 mm, 24 parts, among them J1 Conn_01x05_Male, P1 TC2030-MCP, U1 LDO40LPU33RY, U2 DS18B20, U3 STM32F303CCTx, Y1 16Mhz

Commit message: test
Parts:
- moved Y1 6.10 mm to (153.8, 83.0)
Changed lines of the file:
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@@
   )
   (module Crystal:Crystal_SMD_SeikoEpson_FA238-4Pin_3.2x2.5mm (layer F.Cu)
-    (at 152.84 89.04 180)
+    (at 153.84 83.02 180)
     (descr "crystal Epson Toyocom FA-238 https://support.epson.biz/td/api/doc_check.php?dl=brief_fa-238v_en.pdf, 3.2x2.5mm^2 package")
     (tags "SMD SMT crystal")

Commit message: test
Parts:
- moved C9 32.4 mm to (161.3, 78.7)
- moved U2 30.7 mm to (157.0, 103.1)
- moved C3 25.4 mm to (161.0, 82.5)
- moved C7 20.3 mm to (153.9, 98.8), turned to 270 degrees
- moved L1 20.3 mm to (146.8, 98.8), turned to 270 degrees
- moved D2 19.9 mm to (171.5, 104.4)
- moved C8 17.0 mm to (161.1, 84.6)
- moved R1 13.2 mm to (176.5, 104.1)
- moved P1 11.3 mm to (170.4, 85.1), turned to 180 degrees
- moved J1 10.5 mm to (181.6, 99.6), turned to 180 degrees
- moved Y1 10.2 mm to (151.2, 92.9)
- moved C6 4.88 mm to (150.9, 98.8)
- moved D1 3.92 mm to (176.6, 99.3), turned to 180 degrees
- moved R3 3.87 mm to (172.4, 99.1)
- moved C2 3.27 mm to (170.9, 80.8), turned to 180 degrees
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Routing:
- net +3V3: track 0.00 -> 115.3 mm, vias 0 -> 6
- net ~RESET: track 0.00 -> 28.2 mm, vias 0 -> 2
- net SCL: track 0.00 -> 17.9 mm
- net SDA: track 0.00 -> 17.5 mm
- net Net-(C6-Pad2): track 0.00 -> 14.4 mm
- net temperature: track 0.00 -> 12.8 mm
- net Net-(C10-Pad2): track 0.00 -> 12.2 mm
- net Net-(C5-Pad2): track 0.00 -> 9.05 mm
- net SWDSWO: track 0.00 -> 8.94 mm
- net Net-(R3-Pad1): track 0.00 -> 8.72 mm
- net SWDIO: track 0.00 -> 7.95 mm
- net SWDCLK: track 0.00 -> 6.84 mm
- net GND: track 2.06 -> 8.61 mm, vias 1 -> 21
- net Net-(D2-Pad2): track 0.00 -> 5.56 mm
- net +5V: track 0.00 -> 3.94 mm
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